File: 70cm_preamp.sch (KiCad schematic (older format))
At the start: 14 parts, among them J1 Conn_Coaxial, J2 Conn_Coaxial, U1 TA0693, U2 ADL5523

Commit message: v02
Parts:
- removed U1: TA0693, Filter:TA0693A_HandSolder, symbol Filter:TA0693
- removed U2: ADL5523, Package_CSP:LFCSP-8-1EP_3x2mm_P0.5mm_EP1.6x1.65mm_HandSolder, symbol RF_Amplifier:ADL5523
- added U1: TA0693-Filter, 70cm_preamp:TA0693-Filter, symbol 70cm_preamp:TA0693-Filter
- added U2: ADL5523-RF_Amplifier, 70cm_preamp:LFCSP-8-1EP_3x2mm_P0.5mm_EP1.6x1.65mm, symbol 70cm_preamp:ADL5523-RF_Amplifier
- C1: footprint Capacitor_Tantalum_SMD:CP_EIA-3216-10_Kemet-I -> 70cm_preamp:CP_EIA-3216-10_Kemet-I_Pad1.58x1.35mm_HandSolder
- C2: renamed from C3; footprint Capacitor_SMD:C_0603_1608Metric_Pad1.05x0.95mm_HandSolder -> 70cm_preamp:C_0603_1608Metric_Pad1.05x0.95mm_HandSolder
- C3: renamed from C2; footprint Capacitor_SMD:C_0603_1608Metric_Pad1.05x0.95mm_HandSolder -> 70cm_preamp:C_0603_1608Metric_Pad1.05x0.95mm_HandSolder
- D1: footprint Diode_THT:D_DO-35_SOD27_P7.62mm_Horizontal -> 70cm_preamp:D_0603_1608Metric_Pad1.05x0.95mm_HandSolder
- J1: value Conn_Coaxial -> RF_IN; footprint Connector_Coaxial:BNC_Amphenol_B6252HB-NPP3G-50_Horizontal -> 70cm_preamp:SMA_Amphenol_132289_EdgeMount
- J2: value Conn_Coaxial -> RF_OUT; footprint Connector_Coaxial:SMA_Amphenol_132289_EdgeMount -> 70cm_preamp:SMA_Amphenol_132289_EdgeMount
- L1: renamed from L2; footprint Inductor_SMD:L_0603_1608Metric_Pad1.05x0.95mm_HandSolder -> 70cm_preamp:L_0603_1608Metric_Pad1.05x0.95mm_HandSolder; TME (none) -> CW0603-8.2
- L2: renamed from L3; value 15n -> 12n; footprint Inductor_SMD:L_0603_1608Metric_Pad1.05x0.95mm_HandSolder -> 70cm_preamp:L_0603_1608Metric_Pad1.05x0.95mm_HandSolder; TME (none) -> CW0603-12
- L3: renamed from L1; value 22n -> 220n; footprint Inductor_SMD:L_0603_1608Metric_Pad1.05x0.95mm_HandSolder -> 70cm_preamp:L_0603_1608Metric_Pad1.05x0.95mm_HandSolder; Lomex 93-01-83 -> (none); TME (none) -> LQW18ANR22J00D
- R1: renamed from R3; footprint Resistor_SMD:R_0603_1608Metric_Pad1.05x0.95mm_HandSolder -> 70cm_preamp:R_0603_1608Metric_Pad1.05x0.95mm_HandSolder
- R2: renamed from R1; footprint Resistor_SMD:R_0603_1608Metric_Pad1.05x0.95mm_HandSolder -> 70cm_preamp:R_0603_1608Metric_Pad1.05x0.95mm_HandSolder
- R3: renamed from R2; footprint Resistor_SMD:R_0603_1608Metric_Pad1.05x0.95mm_HandSolder -> 70cm_preamp:SolderJumper-2_P1.3mm_Open_Pad1.0x1.5mm
Connections:
- wire segments 24 -> 45
Other:
- moved on the sheet: C1, C2, C3, D1, J1, J2, L1, L2, L3, R1, R2, R3

Commit message: v02.000001
Parts:
- D1: footprint 70cm_preamp:D_0603_1608Metric_Pad1.05x0.95mm_HandSolder -> 70cm_preamp:D_SOD-123; TME (none) -> CD4148WT(0603C)
- J1, J2: Lomex (none) -> 43-28-28; TME (none) -> RF2-145A-T-17-50-G-HDW
- U1: Farnell (none) -> Alternative (different size!): AFS434S3-T
Changed lines of the file:
@@
 F 1 "RF_OUT" H 7649 3835 50  0000 L CNN
 F 2 "70cm_preamp:SMA_Amphenol_132289_EdgeMount" H 7550 3950 50  0001 C CNN
-F 3 " ~" H 7550 3950 50  0001 C CNN
+F 3 "https://www.tme.eu/Document/b4dd5925cecd78bf6385fa91265dd943/RF2-145A-T-17-50-G-HDW.pdf" H 7550 3950 50  0001 C CNN
+F 4 "43-28-28" H 7550 3950 50  0001 C CNN "Lomex"
+F 5 "RF2-145A-T-17-50-G-HDW " H 7550 3950 50  0001 C CNN "TME"
 	1    7550 3950
 	1    0    0    -1
@@
 F 1 "RF_IN" H 4450 3850 50  0000 C CNN
 F 2 "70cm_preamp:SMA_Amphenol_132289_EdgeMount" H 4250 3950 50  0001 C CNN
-F 3 " ~" H 4250 3950 50  0001 C CNN
+F 3 "https://www.tme.eu/Document/b4dd5925cecd78bf6385fa91265dd943/RF2-145A-T-17-50-G-HDW.pdf" H 4250 3950 50  0001 C CNN
+F 4 "43-28-28" H 4250 3950 50  0001 C CNN "Lomex"
+F 5 "RF2-145A-T-17-50-G-HDW " H 4250 3950 50  0001 C CNN "TME"
 	1    4250 3950
 	-1   0    0    -1
@@
 F 0 "D1" V 4204 3029 50  0000 L CNN
 F 1 "1N4148" V 4295 3029 50  0000 L CNN
-F 2 "70cm_preamp:D_0603_1608Metric_Pad1.05x0.95mm_HandSolder" H 4250 2775 50  0001 C CNN
-F 3 "https://assets.nexperia.com/documents/data-sheet/1N4148_1N4448.pdf" H 4250 2950 50  0001 C CNN
+F 2 "70cm_preamp:D_SOD-123" H 4250 2775 50  0001 C CNN
+F 3 "https://www.tme.eu/Document/8a0f4bd1d0e0495ebb1834ba060fbfa0/CD4148.pdf" H 4250 2950 50  0001 C CNN
+F 4 "CD4148WT(0603C)" H 4250 2950 50  0001 C CNN "TME"
 	1    4250 2950
 	0    1    1    0
@@
 F 2 "70cm_preamp:TA0693-Filter" H 4900 4300 50  0001 C CNN
 F 3 "https://www.taisaw.com/upload/product/TA0693A%20_Rev.1.0_.pdf" H 4950 4400 50  0001 C CNN
+F 4 "Alternative (different size!): AFS434S3-T" H 5350 4050 50  0001 C CNN "Farnell"
 	1    5350 4050
 	1    0    0    -1

Commit message: LM7805 added
Parts:
- added C4: 100n, symbol Device:C
- added U?: LM78M05, Package_TO_SOT_THT:TO-92_Inline, symbol Regulator_Linear:LM78L05_TO92
Connections:
- wire segments 45 -> 50
Other:
- moved on the sheet: C1, C2, C3, D1, J1, J2, L1, L2, L3, R1, R2, R3

Commit message: Bias-Tee
Parts:
- added C? (x2): 100n, symbol Device:C
- added C?: C, symbol Device:C
- added C?: 470u, symbol Device:CP
- added D? (x4): D, symbol Device:D
- added F?: 200mA, symbol Device:Fuse
- added J?: RF, 70cm_preamp:SMA_Amphenol_132289_EdgeMount, symbol Connector:Conn_Coaxial
- added J?: RF+DC, 70cm_preamp:SMA_Amphenol_132289_EdgeMount, symbol Connector:Conn_Coaxial
- added L?: 220n, symbol Device:L
- added P?: Conn_WallPlug_Earth, symbol Connector:Conn_WallPlug_Earth
- added SW?: SW_SPST, symbol Switch:SW_SPST
- added T?: Transformer_1P_1S, symbol Device:Transformer_1P_1S
- added U?: LM7809_TO220, Package_TO_SOT_THT:TO-220-3_Vertical, symbol Regulator_Linear:LM7809_TO220
- D1: TME CD4148WT(0603C) -> (none)
- L3: TME LQW18ANR22J00D -> 0805AS-R22J-08
Connections:
- net labels added: +5V, +9V, GNDA
- wire segments 50 -> 92
Other:
- moved on the sheet: D1, J2, L3, R3

Commit message: Optikai tuning
Parts:
- removed C?: C, symbol Device:C
- removed P?: Conn_WallPlug_Earth, symbol Connector:Conn_WallPlug_Earth
- removed SW?: SW_SPST, symbol Switch:SW_SPST
- added C8: 82p, symbol Device:C
- added J5: 230V AC, symbol 70cm_preamp:Screw_Terminal_01x02
- F1: renamed from F?; value 200mA -> Fuse 200mA
- gave numbers to parts that had none: 13
Connections:
- wire segments 92 -> 89
Other:
- note added: "Erősítő"
- note added: "Tápegység"
- moved on the sheet: C1, C2, C3, C4, C5, C6, C7, D1, J1, J2, J3, J4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

Commit message: RF alkatreszek
Parts:
- added C5: 82p, 70cm_preamp:C_0603_1608Metric_Pad1.05x0.95mm_HandSolder, symbol Device:C
- C4: footprint (none) -> 70cm_preamp:C_0603_1608Metric_Pad1.05x0.95mm_HandSolder
- C6: renamed from C5; footprint (none) -> 70cm_preamp:C_0603_1608Metric_Pad1.05x0.95mm_HandSolder
- C7: renamed from C6; footprint (none) -> 70cm_preamp:C_0603_1608Metric_Pad1.05x0.95mm_HandSolder
- C8: renamed from C7; footprint (none) -> 70cm_preamp:C_0603_1608Metric_Pad1.05x0.95mm_HandSolder
- C9: renamed from C8; footprint (none) -> 70cm_preamp:C_0603_1608Metric_Pad1.05x0.95mm_HandSolder; RF (none) -> RF
- J1, J2: footprint 70cm_preamp:SMA_Amphenol_132289_EdgeMount -> 70cm_preamp:SMA_Amphenol_901-144_Vertical
- L1, L3: RF (none) -> RF
- L4: footprint (none) -> 70cm_preamp:L_0603_1608Metric_Pad1.05x0.95mm_HandSolder; RF (none) -> RF
- renumbered D1 to D5
Connections:
- wire segments 89 -> 90
Other:
- note added: "Dobozok:\n5,1 x 5,1 x 3,2 cm: https://www.tme.eu/hu/details/alu-g0470/univerzalis-keszulekhazak/gainta/g-0470/\n3,8 x 9 x 3 cm: https://www.tme.eu/hu/details/alu-g0123/univerzalis-keszulekhazak/gainta/g-0123/"
Changed lines of the file:
@@
 F 0 "J2" H 8149 2326 50  0000 L CNN
 F 1 "RF_OUT" H 8149 2235 50  0000 L CNN
-F 2 "70cm_preamp:SMA_Amphenol_132289_EdgeMount" H 8050 2350 50  0001 C CNN
+F 2 "70cm_preamp:SMA_Amphenol_901-144_Vertical" H 8050 2350 50  0001 C CNN
 F 3 "https://www.tme.eu/Document/b4dd5925cecd78bf6385fa91265dd943/RF2-145A-T-17-50-G-HDW.pdf" H 8050 2350 50  0001 C CNN
 F 4 "43-28-28" H 8050 2350 50  0001 C CNN "Lomex"
@@
 F 4 "93-02-56" V 4900 2350 50  0001 C CNN "Lomex"
 F 5 "CW0603-8.2" H 4900 2350 50  0001 C CNN "TME"
+F 6 "RF" V 4800 2350 50  0000 C CNN "RF"
 	1    4900 2350
 	0    -1   -1   0
@@
 F 0 "J1" H 3500 2350 50  0000 C CNN
 F 1 "RF_IN" H 3450 2250 50  0000 C CNN
-F 2 "70cm_preamp:SMA_Amphenol_132289_EdgeMount" H 3250 2350 50  0001 C CNN
+F 2 "70cm_preamp:SMA_Amphenol_901-144_Vertical" H 3250 2350 50  0001 C CNN
 F 3 "https://www.tme.eu/Document/b4dd5925cecd78bf6385fa91265dd943/RF2-145A-T-17-50-G-HDW.pdf" H 3250 2350 50  0001 C CNN
 F 4 "43-28-28" H 3250 2350 50  0001 C CNN "Lomex"
@@
 F 4 "" H 7450 1950 50  0001 C CNN "Lomex"
 F 5 " 0805AS-R22J-08" H 7450 1950 50  0001 C CNN "TME"
+F 6 "RF" H 7350 1950 50  0000 C CNN "RF"
 	1    7450 1950
 	1    0    0    -1
@@
 $EndComp
 $Comp
-L Diode:1N4148 D1
+L Diode:1N4148 D5
 U 1 1 5DF6CDEB
 P 7000 1350
-F 0 "D1" V 6954 1429 50  0000 L CNN
+F 0 "D5" V 6954 1429 50  0000 L CNN
 F 1 "1N4148" V 7045 1429 50  0000 L CNN
 F 2 "70cm_preamp:D_SOD-123" H 7000 1175 50  0001 C CNN
@@
 Connection ~ 5350 1100
 $Comp
-L power:GND #PWR?
+L power:GND #PWR0103
 U 1 1 601C2946
 P 6050 1600
-F 0 "#PWR?" H 6050 1350 50  0001 C CNN
+F 0 "#PWR0103" H 6050 1350 50  0001 C CNN
 F 1 "GND" H 6055 1427 50  0000 C CNN
 F 2 "" H 6050 1600 50  0001 C CNN
@@
 F 0 "C4" H 6665 1396 50  0000 L CNN
 F 1 "100n" H 6665 1305 50  0000 L CNN
-F 2 "" H 6588 1200 50  0001 C CNN
+F 2 "70cm_preamp:C_0603_1608Metric_Pad1.05x0.95mm_HandSolder" H 6588 1200 50  0001 C CNN
 F 3 "~" H 6550 1350 50  0001 C CNN
 	1    6550 1350
@@
 	6550 1100 6350 1100
 $Comp
-L power:GND #PWR?
+L power:GND #PWR0104
 U 1 1 601F7623
 P 6550 1600
-F 0 "#PWR?" H 6550 1350 50  0001 C CNN
+F 0 "#PWR0104" H 6550 1350 50  0001 C CNN
 F 1 "GND" H 6555 1427 50  0000 C CNN
 F 2 "" H 6550 1600 50  0001 C CNN
@@
 $EndComp
 $Comp
-L Device:C C6
+L Device:C C7
 U 1 1 601C18DD
 P 6000 4950
-F 0 "C6" H 6115 4996 50  0000 L CNN
+F 0 "C7" H 6115 4996 50  0000 L CNN
 F 1 "100n" H 6115 4905 50  0000 L CNN
-F 2 "" H 6038 4800 50  0001 C CNN
+F 2 "70cm_preamp:C_0603_1608Metric_Pad1.05x0.95mm_HandSolder" H 6038 4800 50  0001 C CNN
 F 3 "~" H 6000 4950 50  0001 C CNN
 	1    6000 4950
@@
 	6000 4600 6250 4600
 $Comp
-L power:GNDA #PWR?
+L power:GNDA #PWR0105
 U 1 1 601D7D5D
 P 4700 6100
-F 0 "#PWR?" H 4700 5850 50  0001 C CNN
+F 0 "#PWR0105" H 4700 5850 50  0001 C CNN
 F 1 "GNDA" H 4705 5927 50  0000 C CNN
 F 2 "" H 4700 6100 50  0001 C CNN
@@
 $EndComp
 $Comp
-L Device:C C7
+L Device:C C8
 U 1 1 601D8420
 P 7100 4950
-F 0 "C7" H 7215 4996 50  0000 L CNN
+F 0 "C8" H 7215 4996 50  0000 L CNN
 F 1 "100n" H 7215 4905 50  0000 L CNN
-F 2 "" H 7138 4800 50  0001 C CNN
+F 2 "70cm_preamp:C_0603_1608Metric_Pad1.05x0.95mm_HandSolder" H 7138 4800 50  0001 C CNN
 F 3 "~" H 7100 4950 50  0001 C CNN
 	1    7100 4950
@@
 $EndComp
 $Comp
-L power:GNDA #PWR?
+L power:GNDA #PWR0106
 U 1 1 601E39A7
 P 6000 5200
-F 0 "#PWR?" H 6000 4950 50  0001 C CNN
+F 0 "#PWR0106" H 6000 4950 50  0001 C CNN
 F 1 "GNDA" H 6005 5027 50  0000 C CNN
 F 2 "" H 6000 5200 50  0001 C CNN
@@
 $EndComp
 $Comp
-L power:GNDA #PWR?
+L power:GNDA #PWR0107
 U 1 1 601E3D51
 P 6550 5200
-F 0 "#PWR?" H 6550 4950 50  0001 C CNN
+F 0 "#PWR0107" H 6550 4950 50  0001 C CNN
 F 1 "GNDA" H 6555 5027 50  0000 C CNN
 F 2 "" H 6550 5200 50  0001 C CNN
@@
 	6000 5100 6000 5200
 $Comp
-L power:GNDA #PWR?
+L power:GNDA #PWR0108
 U 1 1 601E8368
 P 7100 5200
-F 0 "#PWR?" H 7100 4950 50  0001 C CNN
+F 0 "#PWR0108" H 7100 4950 50  0001 C CNN
 F 1 "GNDA" H 7105 5027 50  0000 C CNN
 F 2 "" H 7100 5200 50  0001 C CNN
@@
 	7100 5200 7100 5100
 $Comp
-L power:+9V #PWR?
+L power:+9V #PWR0109
 U 1 1 601F6885
 P 7100 4500
-F 0 "#PWR?" H 7100 4350 50  0001 C CNN
+F 0 "#PWR0109" H 7100 4350 50  0001 C CNN
 F 1 "+9V" H 7115 4673 50  0000 C CNN
 F 2 "" H 7100 4500 50  0001 C CNN
@@
 Connection ~ 7100 4600
 $Comp
-L power:+5V #PWR?
+L power:+5V #PWR0110
 U 1 1 60203FDC
 P 5350 1000
-F 0 "#PWR?" H 5350 850 50  0001 C CNN
+F 0 "#PWR0110" H 5350 850 50  0001 C CNN
 F 1 "+5V" H 5365 1173 50  0000 C CNN
 F 2 "" H 5350 1000 50  0001 C CNN
@@
 F 0 "L4" V 7640 4600 50  0000 C CNN
 F 1 "220n" V 7549 4600 50  0000 C CNN
-F 2 "" H 7450 4600 50  0001 C CNN
+F 2 "70cm_preamp:L_0603_1608Metric_Pad1.05x0.95mm_HandSolder" H 7450 4600 50  0001 C CNN
 F 3 "https://www.tme.eu/hu/details/0805as-r22j-08/smd-0805-induktorok/fastron/" H 7450 4600 50  0001 C CNN
 F 4 " 0805AS-R22J-08" H 7450 4600 50  0001 C CNN "TME"
+F 5 "RF" V 7350 4600 50  0000 C CNN "RF"
 	1    7450 4600
 	0    -1   -1   0
@@
 Connection ~ 7800 4600
 $Comp
-L power:GNDA #PWR?
+L power:GNDA #PWR0111
 U 1 1 6022329F
 P 8000 5450
-F 0 "#PWR?" H 8000 5200 50  0001 C CNN
+F 0 "#PWR0111" H 8000 5200 50  0001 C CNN
 F 1 "GNDA" H 8005 5277 50  0000 C CNN
 F 2 "" H 8000 5450 50  0001 C CNN
@@
 $EndComp
 $Comp
-L power:GNDA #PWR?
+L power:GNDA #PWR0112
 U 1 1 60226CA6
 P 8000 4100
-F 0 "#PWR?" H 8000 3850 50  0001 C CNN
+F 0 "#PWR0112" H 8000 3850 50  0001 C CNN
 F 1 "GNDA" H 8005 3927 50  0000 C CNN
 F 2 "" H 8000 4100 50  0001 C CNN
@@
 $EndComp
 $Comp
-L Device:CP C5
+L Device:CP C6
 U 1 1 60233EE0
 P 5300 4950
-F 0 "C5" H 5418 4996 50  0000 L CNN
+F 0 "C6" H 5418 4996 50  0000 L CNN
 F 1 "470u" H 5418 4905 50  0000 L CNN
-F 2 "" H 5338 4800 50  0001 C CNN
+F 2 "70cm_preamp:C_0603_1608Metric_Pad1.05x0.95mm_HandSolder" H 5338 4800 50  0001 C CNN
 F 3 "~" H 5300 4950 50  0001 C CNN
 	1    5300 4950
@@
 	5300 5100 5300 5200
 $Comp
-L power:GNDA #PWR?
+L power:GNDA #PWR0113
 U 1 1 6025C01D
 P 5300 5200
-F 0 "#PWR?" H 5300 4950 50  0001 C CNN
+F 0 "#PWR0113" H 5300 4950 50  0001 C CNN
 F 1 "GNDA" H 5305 5027 50  0000 C CNN
 F 2 "" H 5300 5200 50  0001 C CNN
@@
 	7000 1100 7450 1100
 Wire Wire Line
-	5750 2350 7450 2350
+	5750 2350 6850 2350
 $Comp
 L Device:D D2
@@
 Tápegység
 $Comp
-L Device:C C8
+L Device:C C9
 U 1 1 60397086
 P 7800 4950
-F 0 "C8" H 7915 4996 50  0000 L CNN
+F 0 "C9" H 7915 4996 50  0000 L CNN
 F 1 "82p" H 7915 4905 50  0000 L CNN
-F 2 "" H 7838 4800 50  0001 C CNN
+F 2 "70cm_preamp:C_0603_1608Metric_Pad1.05x0.95mm_HandSolder" H 7838 4800 50  0001 C CNN
 F 3 "~" H 7800 4950 50  0001 C CNN
+F 4 "RF" H 7650 4950 50  0000 C CNN "RF"
 	1    7800 4950
 	1    0    0    -1
@@
 	-1   0    0    -1
 $EndComp
+Text Notes 650  7650 0    50   ~ 0
+Dobozok:\n5,1 x 5,1 x 3,2 cm: https://www.tme.eu/hu/details/alu-g0470/univerzalis-keszulekhazak/gainta/g-0470/\n3,8 x 9 x 3 cm: https://www.tme.eu/hu/details/alu-g0123/univerzalis-keszulekhazak/gainta/g-0123/
+$Comp
+L Device:C C5
+U 1 1 602B5DC9
+P 7000 2350
+F 0 "C5" V 6750 2300 50  0000 L CNN
+F 1 "82p" V 6850 2300 50  0000 L CNN
+F 2 "70cm_preamp:C_0603_1608Metric_Pad1.05x0.95mm_HandSolder" H 7038 2200 50  0001 C CNN
+F 3 "~" H 7000 2350 50  0001 C CNN
+F 4 "RF" V 7150 2350 50  0000 C CNN "RF"
+	1    7000 2350
+	0    1    1    0
+$EndComp
+Wire Wire Line
+	7150 2350 7450 2350
 $EndSCHEMATC

Commit message: rajzolatok
Parts:
- removed C1: 1u, 70cm_preamp:CP_EIA-3216-10_Kemet-I_Pad1.58x1.35mm_HandSolder, symbol Device:CP
- removed C2, C4: 100n, 70cm_preamp:C_0603_1608Metric_Pad1.05x0.95mm_HandSolder, symbol Device:C
- removed C3: 100p, 70cm_preamp:C_0603_1608Metric_Pad1.05x0.95mm_HandSolder, symbol Device:C
- removed D5: 1N4148, 70cm_preamp:D_SOD-123, symbol Diode:1N4148
- removed L1: 8n2, 70cm_preamp:L_0603_1608Metric_Pad1.05x0.95mm_HandSolder, symbol Device:L
- removed L2: 12n, 70cm_preamp:L_0603_1608Metric_Pad1.05x0.95mm_HandSolder, symbol Device:L
- removed R1: 10k, 70cm_preamp:R_0603_1608Metric_Pad1.05x0.95mm_HandSolder, symbol Device:R
- removed R2: 1k3, 70cm_preamp:R_0603_1608Metric_Pad1.05x0.95mm_HandSolder, symbol Device:R
- removed U1: TA0693-Filter, 70cm_preamp:TA0693-Filter, symbol 70cm_preamp:TA0693-Filter
- removed U2: ADL5523-RF_Amplifier, 70cm_preamp:LFCSP-8-1EP_3x2mm_P0.5mm_EP1.6x1.65mm, symbol 70cm_preamp:ADL5523-RF_Amplifier
- removed U4: LM7809_TO220, Package_TO_SOT_THT:TO-220-3_Vertical, symbol Regulator_Linear:LM7809_TO220
- added U?: PGA-103+, 70cm_preamp:SOT-89-3, symbol 70cm_preamp:PGA-103+
- added U?: SF2446E, Filter:TA0693A, symbol 70cm_preamp:SF2446E
Connections:
- wire segments 90 -> 57
Other:
- moved on the sheet: C5, J1, J2, L3, R3

Commit message: nyák
Parts:
- removed C5: 82p, 70cm_preamp:C_0603_1608Metric_Pad1.05x0.95mm_HandSolder, symbol Device:C
- removed L3: 220n, 70cm_preamp:L_0603_1608Metric_Pad1.05x0.95mm_HandSolder, symbol Device:L
- removed R3: 0, 70cm_preamp:SolderJumper-2_P1.3mm_Open_Pad1.0x1.5mm, symbol Device:R
- D1, D2, D3, D4: footprint (none) -> 70cm_preamp:D_SOD-123
- U1: renamed from U?; footprint Filter:TA0693A -> 70cm_preamp:SF2446E-Filter_Custom_HandSolder
- gave numbers to parts that had none: 1
- renumbered C6 to C1, C7 to C2, C8 to C3, C9 to C4, L4 to L1
Connections:
- net labels removed: +5V
- wire segments 57 -> 52
Other:
- moved on the sheet: J1, J2
