File: 70cm_preamp.sch (KiCad schematic (older format))
At the start: 19 parts, among them J1 RF_IN, J2 RF_OUT, J3 RF+DC, J4 RF, J5 230V AC, T1 Transformer_1P_1S, U1 SF2446E, U2 PGA-103+, U3 LM78M05

Commit message: Stabilitáshoz RLC
Parts:
- added C1: 330p, 70cm_preamp:C_0603_1608Metric_Pad1.05x0.95mm_HandSolder, symbol Device:C
- added L1: 620n, 70cm_preamp:L_0603_1608Metric_Pad1.05x0.95mm_HandSolder, symbol Device:L
- added R1: 150, 70cm_preamp:R_0603_1608Metric_Pad1.05x0.95mm_HandSolder, symbol Device:R
- renumbered C1 to C2, C2 to C3, C3 to C4, C4 to C5, L1 to L2
Connections:
- wire segments 52 -> 55
Other:
- moved on the sheet: J1, J2
Changed lines of the file:
@@
 L Connector:Conn_Coaxial J2
 U 1 1 5DF66D76
-P 7050 1850
-F 0 "J2" H 7149 1826 50  0000 L CNN
-F 1 "RF_OUT" H 7149 1735 50  0000 L CNN
-F 2 "70cm_preamp:SMA_Amphenol_901-144_Vertical" H 7050 1850 50  0001 C CNN
-F 3 "https://www.tme.eu/Document/b4dd5925cecd78bf6385fa91265dd943/RF2-145A-T-17-50-G-HDW.pdf" H 7050 1850 50  0001 C CNN
-F 4 "43-28-28" H 7050 1850 50  0001 C CNN "Lomex"
-F 5 "RF2-145A-T-17-50-G-HDW " H 7050 1850 50  0001 C CNN "TME"
-	1    7050 1850
+P 7500 1850
+F 0 "J2" H 7599 1826 50  0000 L CNN
+F 1 "RF_OUT" H 7599 1735 50  0000 L CNN
+F 2 "70cm_preamp:SMA_Amphenol_901-144_Vertical" H 7500 1850 50  0001 C CNN
+F 3 "https://www.tme.eu/Document/b4dd5925cecd78bf6385fa91265dd943/RF2-145A-T-17-50-G-HDW.pdf" H 7500 1850 50  0001 C CNN
+F 4 "43-28-28" H 7500 1850 50  0001 C CNN "Lomex"
+F 5 "RF2-145A-T-17-50-G-HDW " H 7500 1850 50  0001 C CNN "TME"
+	1    7500 1850
 	1    0    0    -1
 $EndComp
@@
 L power:GND #PWR07
 U 1 1 5DF66E82
-P 7050 2400
-F 0 "#PWR07" H 7050 2150 50  0001 C CNN
-F 1 "GND" H 7055 2227 50  0000 C CNN
-F 2 "" H 7050 2400 50  0001 C CNN
-F 3 "" H 7050 2400 50  0001 C CNN
-	1    7050 2400
+P 7500 2850
+F 0 "#PWR07" H 7500 2600 50  0001 C CNN
+F 1 "GND" H 7505 2677 50  0000 C CNN
+F 2 "" H 7500 2850 50  0001 C CNN
+F 3 "" H 7500 2850 50  0001 C CNN
+	1    7500 2850
 	1    0    0    -1
 $EndComp
@@
 L Connector:Conn_Coaxial J1
 U 1 1 5DF686B1
-P 4200 1850
-F 0 "J1" H 4450 1850 50  0000 C CNN
-F 1 "RF_IN" H 4400 1750 50  0000 C CNN
-F 2 "70cm_preamp:SMA_Amphenol_901-144_Vertical" H 4200 1850 50  0001 C CNN
-F 3 "https://www.tme.eu/Document/b4dd5925cecd78bf6385fa91265dd943/RF2-145A-T-17-50-G-HDW.pdf" H 4200 1850 50  0001 C CNN
-F 4 "43-28-28" H 4200 1850 50  0001 C CNN "Lomex"
-F 5 "RF2-145A-T-17-50-G-HDW " H 4200 1850 50  0001 C CNN "TME"
-	1    4200 1850
+P 3850 1850
+F 0 "J1" H 4100 1850 50  0000 C CNN
+F 1 "RF_IN" H 4050 1750 50  0000 C CNN
+F 2 "70cm_preamp:SMA_Amphenol_901-144_Vertical" H 3850 1850 50  0001 C CNN
+F 3 "https://www.tme.eu/Document/b4dd5925cecd78bf6385fa91265dd943/RF2-145A-T-17-50-G-HDW.pdf" H 3850 1850 50  0001 C CNN
+F 4 "43-28-28" H 3850 1850 50  0001 C CNN "Lomex"
+F 5 "RF2-145A-T-17-50-G-HDW " H 3850 1850 50  0001 C CNN "TME"
+	1    3850 1850
 	-1   0    0    -1
 $EndComp
@@
 L power:GND #PWR01
 U 1 1 5DF68779
-P 4200 2400
-F 0 "#PWR01" H 4200 2150 50  0001 C CNN
-F 1 "GND" H 4205 2227 50  0000 C CNN
-F 2 "" H 4200 2400 50  0001 C CNN
-F 3 "" H 4200 2400 50  0001 C CNN
-	1    4200 2400
-	1    0    0    -1
-$EndComp
-Wire Wire Line
-	4200 2400 4200 2050
-Wire Wire Line
-	7050 2400 7050 2050
+P 3850 2850
+F 0 "#PWR01" H 3850 2600 50  0001 C CNN
+F 1 "GND" H 3855 2677 50  0000 C CNN
+F 2 "" H 3850 2850 50  0001 C CNN
+F 3 "" H 3850 2850 50  0001 C CNN
+	1    3850 2850
+	1    0    0    -1
+$EndComp
 $Comp
 L Regulator_Linear:LM78L05_TO92 U3
@@
 $EndComp
 $Comp
-L Device:C C2
+L Device:C C3
 U 1 1 601C18DD
 P 6000 4950
-F 0 "C2" H 6115 4996 50  0000 L CNN
+F 0 "C3" H 6115 4996 50  0000 L CNN
 F 1 "100n" H 6115 4905 50  0000 L CNN
 F 2 "70cm_preamp:C_0603_1608Metric_Pad1.05x0.95mm_HandSolder" H 6038 4800 50  0001 C CNN
@@
 $EndComp
 $Comp
-L Device:C C3
+L Device:C C4
 U 1 1 601D8420
 P 7100 4950
-F 0 "C3" H 7215 4996 50  0000 L CNN
+F 0 "C4" H 7215 4996 50  0000 L CNN
 F 1 "100n" H 7215 4905 50  0000 L CNN
 F 2 "70cm_preamp:C_0603_1608Metric_Pad1.05x0.95mm_HandSolder" H 7138 4800 50  0001 C CNN
@@
 Connection ~ 7100 4600
 $Comp
-L Device:L L1
+L Device:L L2
 U 1 1 6021555C
 P 7450 4600
-F 0 "L1" V 7640 4600 50  0000 C CNN
+F 0 "L2" V 7640 4600 50  0000 C CNN
 F 1 "220n" V 7549 4600 50  0000 C CNN
 F 2 "70cm_preamp:L_0603_1608Metric_Pad1.05x0.95mm_HandSolder" H 7450 4600 50  0001 C CNN
@@
 $EndComp
 $Comp
-L Device:CP C1
+L Device:CP C2
 U 1 1 60233EE0
 P 5300 4950
-F 0 "C1" H 5418 4996 50  0000 L CNN
+F 0 "C2" H 5418 4996 50  0000 L CNN
 F 1 "470u" H 5418 4905 50  0000 L CNN
 F 2 "70cm_preamp:C_0603_1608Metric_Pad1.05x0.95mm_HandSolder" H 5338 4800 50  0001 C CNN
@@
 Tápegység
 $Comp
-L Device:C C4
+L Device:C C5
 U 1 1 60397086
 P 7800 4950
-F 0 "C4" H 7915 4996 50  0000 L CNN
+F 0 "C5" H 7915 4996 50  0000 L CNN
 F 1 "82p" H 7915 4905 50  0000 L CNN
 F 2 "70cm_preamp:C_0603_1608Metric_Pad1.05x0.95mm_HandSolder" H 7838 4800 50  0001 C CNN
@@
 L 70cm_preamp:PGA-103+ U2
 U 1 1 60481085
-P 6000 1850
-F 0 "U2" H 6050 2215 50  0000 C CNN
-F 1 "PGA-103+" H 6050 2124 50  0000 C CNN
-F 2 "70cm_preamp:SOT-89-3" H 5600 2050 50  0001 C CNN
-F 3 "https://www.minicircuits.com/pdfs/PGA-103+.pdf" H 5700 2150 50  0001 C CNN
-	1    6000 1850
+P 6450 1850
+F 0 "U2" H 6500 2215 50  0000 C CNN
+F 1 "PGA-103+" H 6500 2124 50  0000 C CNN
+F 2 "70cm_preamp:SOT-89-3" H 6050 2050 50  0001 C CNN
+F 3 "https://www.minicircuits.com/pdfs/PGA-103+.pdf" H 6150 2150 50  0001 C CNN
+	1    6450 1850
 	1    0    0    -1
 $EndComp
@@
 L 70cm_preamp:SF2446E U1
 U 1 1 604815FC
-P 4950 1950
-F 0 "U1" H 4950 2275 50  0000 C CNN
-F 1 "SF2446E" H 4950 2184 50  0000 C CNN
-F 2 "70cm_preamp:SF2446E-Filter_Custom_HandSolder" H 4500 2200 50  0001 C CNN
-F 3 "https://wireless.murata.com/datasheet?/RFM/data/sf2446e.pdf" H 4550 2300 50  0001 C CNN
-	1    4950 1950
-	1    0    0    -1
-$EndComp
-Wire Wire Line
-	4650 1850 4400 1850
+P 4600 1950
+F 0 "U1" H 4600 2275 50  0000 C CNN
+F 1 "SF2446E" H 4600 2184 50  0000 C CNN
+F 2 "70cm_preamp:SF2446E-Filter_Custom_HandSolder" H 4150 2200 50  0001 C CNN
+F 3 "https://wireless.murata.com/datasheet?/RFM/data/sf2446e.pdf" H 4200 2300 50  0001 C CNN
+	1    4600 1950
+	1    0    0    -1
+$EndComp
+Wire Wire Line
+	4300 1850 4050 1850
 $Comp
 L power:GND #PWR0101
 U 1 1 60486617
-P 4550 2400
-F 0 "#PWR0101" H 4550 2150 50  0001 C CNN
-F 1 "GND" H 4555 2227 50  0000 C CNN
-F 2 "" H 4550 2400 50  0001 C CNN
-F 3 "" H 4550 2400 50  0001 C CNN
-	1    4550 2400
+P 4200 2850
+F 0 "#PWR0101" H 4200 2600 50  0001 C CNN
+F 1 "GND" H 4205 2677 50  0000 C CNN
+F 2 "" H 4200 2850 50  0001 C CNN
+F 3 "" H 4200 2850 50  0001 C CNN
+	1    4200 2850
 	1    0    0    -1
 $EndComp
@@
 L power:GND #PWR0102
 U 1 1 60486FF7
-P 5350 2400
-F 0 "#PWR0102" H 5350 2150 50  0001 C CNN
-F 1 "GND" H 5355 2227 50  0000 C CNN
-F 2 "" H 5350 2400 50  0001 C CNN
-F 3 "" H 5350 2400 50  0001 C CNN
-	1    5350 2400
-	1    0    0    -1
-$EndComp
-Wire Wire Line
-	4650 2100 4550 2100
-Wire Wire Line
-	4550 2100 4550 2200
-Wire Wire Line
-	4650 2200 4550 2200
-Connection ~ 4550 2200
-Wire Wire Line
-	4550 2200 4550 2400
-Wire Wire Line
-	5250 2100 5350 2100
-Wire Wire Line
-	5350 2100 5350 2200
-Wire Wire Line
-	5250 2200 5350 2200
-Connection ~ 5350 2200
-Wire Wire Line
-	5350 2200 5350 2400
+P 5000 2850
+F 0 "#PWR0102" H 5000 2600 50  0001 C CNN
+F 1 "GND" H 5005 2677 50  0000 C CNN
+F 2 "" H 5000 2850 50  0001 C CNN
+F 3 "" H 5000 2850 50  0001 C CNN
+	1    5000 2850
+	1    0    0    -1
+$EndComp
+Wire Wire Line
+	4300 2100 4200 2100
+Wire Wire Line
+	4200 2100 4200 2200
+Wire Wire Line
+	4300 2200 4200 2200
+Wire Wire Line
+	4900 2100 5000 2100
+Wire Wire Line
+	5000 2100 5000 2200
+Wire Wire Line
+	4900 2200 5000 2200
 $Comp
 L power:GND #PWR0103
 U 1 1 6048CBB9
-P 5950 2400
-F 0 "#PWR0103" H 5950 2150 50  0001 C CNN
-F 1 "GND" H 5955 2227 50  0000 C CNN
-F 2 "" H 5950 2400 50  0001 C CNN
-F 3 "" H 5950 2400 50  0001 C CNN
-	1    5950 2400
-	1    0    0    -1
-$EndComp
-Wire Wire Line
-	5950 2100 5950 2400
-Wire Wire Line
-	5250 1850 5750 1850
-Wire Wire Line
-	6350 1850 6850 1850
+P 6400 2850
+F 0 "#PWR0103" H 6400 2600 50  0001 C CNN
+F 1 "GND" H 6405 2677 50  0000 C CNN
+F 2 "" H 6400 2850 50  0001 C CNN
+F 3 "" H 6400 2850 50  0001 C CNN
+	1    6400 2850
+	1    0    0    -1
+$EndComp
+Wire Wire Line
+	6800 1850 7300 1850
+$Comp
+L Device:L L1
+U 1 1 6050AD32
+P 5650 2050
+F 0 "L1" H 5702 2096 50  0000 L CNN
+F 1 "620n" H 5702 2005 50  0000 L CNN
+F 2 "70cm_preamp:L_0603_1608Metric_Pad1.05x0.95mm_HandSolder" H 5650 2050 50  0001 C CNN
+F 3 "~" H 5650 2050 50  0001 C CNN
+	1    5650 2050
+	1    0    0    -1
+$EndComp
+$Comp
+L Device:R R1
+U 1 1 6050B70A
+P 5650 2350
+F 0 "R1" H 5720 2396 50  0000 L CNN
+F 1 "150" H 5720 2305 50  0000 L CNN
+F 2 "70cm_preamp:R_0603_1608Metric_Pad1.05x0.95mm_HandSolder" V 5580 2350 50  0001 C CNN
+F 3 "~" H 5650 2350 50  0001 C CNN
+	1    5650 2350
+	1    0    0    -1
+$EndComp
+$Comp
+L Device:C C1
+U 1 1 6050BB40
+P 5650 2650
+F 0 "C1" H 5765 2696 50  0000 L CNN
+F 1 "330p" H 5765 2605 50  0000 L CNN
+F 2 "70cm_preamp:C_0603_1608Metric_Pad1.05x0.95mm_HandSolder" H 5688 2500 50  0001 C CNN
+F 3 "~" H 5650 2650 50  0001 C CNN
+	1    5650 2650
+	1    0    0    -1
+$EndComp
+$Comp
+L power:GND #PWR0104
+U 1 1 6050BF6E
+P 5650 2850
+F 0 "#PWR0104" H 5650 2600 50  0001 C CNN
+F 1 "GND" H 5655 2677 50  0000 C CNN
+F 2 "" H 5650 2850 50  0001 C CNN
+F 3 "" H 5650 2850 50  0001 C CNN
+	1    5650 2850
+	1    0    0    -1
+$EndComp
+Connection ~ 4200 2200
+Connection ~ 5000 2200
+Wire Wire Line
+	4900 1850 5650 1850
+Wire Wire Line
+	5650 1900 5650 1850
+Connection ~ 5650 1850
+Wire Wire Line
+	5650 1850 6200 1850
+Wire Wire Line
+	3850 2050 3850 2850
+Wire Wire Line
+	4200 2200 4200 2850
+Wire Wire Line
+	5000 2200 5000 2850
+Wire Wire Line
+	5650 2800 5650 2850
+Wire Wire Line
+	6400 2100 6400 2850
+Wire Wire Line
+	7500 2050 7500 2850
 $EndSCHEMATC

Commit message: 0805 RLC
Parts:
- C1: footprint 70cm_preamp:C_0603_1608Metric_Pad1.05x0.95mm_HandSolder -> 70cm_preamp:C_0805_2012Metric_Pad1.15x1.40mm_HandSolder
- L1: footprint 70cm_preamp:L_0603_1608Metric_Pad1.05x0.95mm_HandSolder -> 70cm_preamp:L_0805_2012Metric_Pad1.15x1.40mm_HandSolder
- R1: footprint 70cm_preamp:R_0603_1608Metric_Pad1.05x0.95mm_HandSolder -> 70cm_preamp:R_0805_2012Metric_Pad1.15x1.40mm_HandSolder
Changed lines of the file:
@@
 F 0 "L1" H 5702 2096 50  0000 L CNN
 F 1 "620n" H 5702 2005 50  0000 L CNN
-F 2 "70cm_preamp:L_0603_1608Metric_Pad1.05x0.95mm_HandSolder" H 5650 2050 50  0001 C CNN
+F 2 "70cm_preamp:L_0805_2012Metric_Pad1.15x1.40mm_HandSolder" H 5650 2050 50  0001 C CNN
 F 3 "~" H 5650 2050 50  0001 C CNN
 	1    5650 2050
@@
 F 0 "R1" H 5720 2396 50  0000 L CNN
 F 1 "150" H 5720 2305 50  0000 L CNN
-F 2 "70cm_preamp:R_0603_1608Metric_Pad1.05x0.95mm_HandSolder" V 5580 2350 50  0001 C CNN
+F 2 "70cm_preamp:R_0805_2012Metric_Pad1.15x1.40mm_HandSolder" V 5580 2350 50  0001 C CNN
 F 3 "~" H 5650 2350 50  0001 C CNN
 	1    5650 2350
@@
 F 0 "C1" H 5765 2696 50  0000 L CNN
 F 1 "330p" H 5765 2605 50  0000 L CNN
-F 2 "70cm_preamp:C_0603_1608Metric_Pad1.05x0.95mm_HandSolder" H 5688 2500 50  0001 C CNN
+F 2 "70cm_preamp:C_0805_2012Metric_Pad1.15x1.40mm_HandSolder" H 5688 2500 50  0001 C CNN
 F 3 "~" H 5650 2650 50  0001 C CNN
 	1    5650 2650

Commit message: Zárójelentés
Other:
- note removed: "Dobozok:\n5,1 x 5,1 x 3,2 cm: https://www.tme.eu/hu/details/alu-g0470/univerzalis-keszulekhazak/gainta/g-0470/\n3,8 x 9 x 3 cm: https://www.tme.eu/hu/details/alu-g0123/univerzalis-keszulekhazak/gainta/g-0123/"
Changed lines of the file:
@@
 	-1   0    0    -1
 $EndComp
-Text Notes 650  7650 0    50   ~ 0
-Dobozok:\n5,1 x 5,1 x 3,2 cm: https://www.tme.eu/hu/details/alu-g0470/univerzalis-keszulekhazak/gainta/g-0470/\n3,8 x 9 x 3 cm: https://www.tme.eu/hu/details/alu-g0123/univerzalis-keszulekhazak/gainta/g-0123/
 $Comp
 L 70cm_preamp:PGA-103+ U2
