File: 70cm_preamp.kicad_pcb (KiCad board)
At the start: 2 copper layers, 37.8 x 15.8 mm, 14 parts, among them J1 Conn_Coaxial, J2 Conn_Coaxial, U1 TA0693, U2 ADL5523

Commit message: nyák
Parts:
- removed C1: 1u, Capacitor_Tantalum_SMD:CP_EIA-3216-10_Kemet-I
- removed C2: 100p, Capacitor_SMD:C_0603_1608Metric_Pad1.05x0.95mm_HandSolder
- removed C3: 100n, Capacitor_SMD:C_0603_1608Metric_Pad1.05x0.95mm_HandSolder
- removed D1: 1N4148, Diode_THT:D_DO-35_SOD27_P7.62mm_Horizontal
- removed L1: 22n, Inductor_SMD:L_0603_1608Metric_Pad1.05x0.95mm_HandSolder
- removed L2: 8n2, Inductor_SMD:L_0603_1608Metric_Pad1.05x0.95mm_HandSolder
- removed L3: 15n, Inductor_SMD:L_0603_1608Metric_Pad1.05x0.95mm_HandSolder
- removed R1: 1k3, Resistor_SMD:R_0603_1608Metric_Pad1.05x0.95mm_HandSolder
- removed R2: 0, Resistor_SMD:R_0603_1608Metric_Pad1.05x0.95mm_HandSolder
- removed R3: 10k, Resistor_SMD:R_0603_1608Metric_Pad1.05x0.95mm_HandSolder
- J1: value Conn_Coaxial -> RF_IN; footprint Connector_Coaxial:BNC_Amphenol_B6252HB-NPP3G-50_Horizontal -> 70cm_preamp:SMA_Amphenol_901-144_Vertical; moved to F.Cu
- J2: value Conn_Coaxial -> RF_OUT; footprint Connector_Coaxial:SMA_Amphenol_132289_EdgeMount -> 70cm_preamp:SMA_Amphenol_901-144_Vertical
- U1: value TA0693 -> SF2446E; footprint Filter:TA0693A_HandSolder -> 70cm_preamp:SF2446E-Filter_Custom_HandSolder
- U2: value ADL5523 -> PGA-103+; footprint Package_CSP:LFCSP-8-1EP_3x2mm_P0.5mm_EP1.6x1.65mm_HandSolder -> 70cm_preamp:SOT-89-3
- moved J2 33.3 mm to (32.0, 23.0), turned to 0 degrees
- moved U2 31.2 mm to (42.5, 24.5), turned to 270 degrees
- moved U1 31.0 mm to (51.5, 23.0), turned to 180 degrees
- moved J1 25.8 mm to (62.5, 23.0), turned to 0 degrees
Connections:
- U1 pad 5: GND -> Net-(U1-Pad5)
- U1 pad 6: Net-(L2-Pad1) -> GND
- U2 pad 1: Net-(R1-Pad1) -> Net-(U1-Pad5)
- U2 pad 2: Net-(L2-Pad2) -> GND
- U2 pad 3: (no net) -> Net-(J2-Pad1)
Routing:
- net Net-(C1-Pad1): track 9.18 -> 0.00 mm
- net Net-(U1-Pad5): track 0.00 -> 6.18 mm
- net Net-(R1-Pad1): track 4.90 -> 0.00 mm, vias 2 -> 0
- net Net-(J1-Pad1): track 5.52 -> 9.67 mm
- net Net-(L3-Pad2): track 3.26 -> 0.00 mm
- net Net-(L1-Pad1): track 2.39 -> 0.00 mm
- net Net-(L2-Pad2): track 1.93 -> 0.00 mm
- net Net-(L2-Pad1): track 1.82 -> 0.00 mm
- net Net-(J2-Pad1): track 8.10 -> 9.00 mm
- added copper zone on B.Cu, net GND
Other:
- board outline removed
- net class Tapvonal_50 added: clearance 0.15, trace_width 0.81, via_dia 0.8, via_drill 0.4
- board text removed: "HA5KFU 70cm preamp"

Commit message: nyák
Parts:
- added REF**: SMA_Amphenol_132289_EdgeMount, 70cm_preamp:SMA_Amphenol_132289_EdgeMount, F.Cu at (45.0, 36.8)
- added REF**: SMA_Amphenol_132289_EdgeMount, 70cm_preamp:SMA_Amphenol_132289_EdgeMount, F.Cu at (73.2, 36.8)
- moved J2 20.8 mm to (47.6, 36.8)
- moved U2 19.2 mm to (55.8, 38.3)
- moved U1 17.6 mm to (62.4, 36.8)
- moved J1 16.0 mm to (70.6, 36.8)
Routing:
- net Net-(U1-Pad5): track 6.18 -> 3.78 mm
- net GND: vias 0 -> 44
Other:
- board outline added: 33.4 x 13.2 mm
- net class Tapvonal_50 removed
- net class Tapvonal_vastag added: clearance 0.33, trace_width 1.3, via_dia 0.8, via_drill 0.4
- net class Tapvonal_vekony added: clearance 0.12, trace_width 0.81, via_dia 0.8, via_drill 0.4
- board text added: "70 cm preamp HA5KFU"

Commit message: csak tht sma
Parts:
- removed REF** (x2): SMA_Amphenol_132289_EdgeMount, 70cm_preamp:SMA_Amphenol_132289_EdgeMount
- turned J1 to 270 degrees
Routing:
- net Net-(J2-Pad1): track 9.40 -> 6.70 mm
- net Net-(J1-Pad1): track 9.48 -> 6.87 mm
- net GND: vias 44 -> 28
Other:
- board text added: "ANT"
- board text added: "HA5KFU"
- board text added: "RCV"
- board text removed: "70 cm preamp HA5KFU"
